File: Dash_Warning_Panel.sch (KiCad schematic (older format))
At the start: 29 parts, among them J1 Conn_01x06_Male, SW1 SW_DIP_x02, U1 LP5024, U2 TPS22810-Q1

Commit message: Routing with LP5024
Ready for Fabrication Review
Parts:
- U1: footprint (none) -> Housings_DFN_QFN:QFN-32-1EP_5x5mm_Pitch0.5mm
Changed lines of the file:
@@
 F 0 "U1" H 7250 2500 50  0000 C CNN
 F 1 "LP5024" H 7250 4400 50  0000 C CNN
-F 2 "" H 7250 3450 50  0001 C CNN
+F 2 "Housings_DFN_QFN:QFN-32-1EP_5x5mm_Pitch0.5mm" H 7250 3450 50  0001 C CNN
 F 3 "" H 7250 3450 50  0001 C CNN
 	1    7250 3450
