File: Dash_Warning_Panel.kicad_pcb (KiCad board)
At the start: 2 copper layers, 53 x 40 mm, 43 parts, among them J1 Conn, U1 TLC6C5816, U2 TPS22810, U3 TLV741P

Commit message: Backlog Push
Whatever Changed since 2021
Other:
- rule pad_to_mask_clearance: 0.0508 -> 0
